Commit message: Working SITL

File: uvify_description/xacro/d435.xacro (robot description, xacro)
@@ -8,5 +8,5 @@
 <robot name="sensor_d435" xmlns:xacro="http://ros.org/wiki/xacro">
   <!--File includes-->
-  <xacro:include filename="$(find ifo_description)/xacro/d435.gazebo.xacro"/>
+  <xacro:include filename="$(find uvify_description)/xacro/d435.gazebo.xacro"/>
   <xacro:macro name="sensor_d435" params="name:=camera topics_ns:=camera parent *origin publish_pointcloud:=true">
     <xacro:property name="M_PI" value="3.1415926535897931" />
@@ -45,5 +45,5 @@
         <geometry>
           <!-- <box size="${d435_cam_width} ${d435_cam_height} ${d435_cam_depth}"/> -->
-          <mesh filename="package://ifo_description/meshes/d435.dae" />
+          <mesh filename="package://uvify_description/meshes/d435.dae" />
           <!--<mesh filename="package://realsense2_description/meshes/d435/d435.dae" />-->
         </geometry>

File: uvify_description/xacro/iris.xacro (robot description, xacro)
@@ -2,11 +2,11 @@
 <robot xmlns:xacro="http://www.ros.org/wiki/xacro" name="iris">
   <xacro:macro name="iris_base_macro" params="mavlink_udp_port:=14560 mavlink_tcp_port:=4560 namespace:=default_ns">
-    <xacro:include filename="$(find ifo_description)/materials/materials.xacro" />
+    <xacro:include filename="$(find uvify_description)/materials/materials.xacro" />
     <!-- Base Link: Main Chassis -->
-    <link name="base_link">
+    <link name="${namespace}/base_link">
       <origin xyz="0 0 0" rpy="0 0 0"/>
       <visual>
         <geometry>
-          <mesh filename="package://ifo_description/meshes/iris.stl" />
+          <mesh filename="package://uvify_description/meshes/iris.stl" />
         </geometry>
         <material name="DarkGrey"/>
@@ -38,5 +38,5 @@
       </inertial>
     </link>
-    <gazebo reference="base_link">
+    <gazebo reference="${namespace}/base_link">
       <collision>
         <surface>
@@ -60,8 +60,8 @@
     <!--                               ROTOR 0                                 -->
     <!-- ===================================================================== -->
-    <link name='rotor_0'>
+    <link name='${namespace}/rotor_0'>
       <visual>
         <geometry>
-          <mesh filename="package://ifo_description/meshes/iris_prop_ccw.dae"/>
+          <mesh filename="package://uvify_description/meshes/iris_prop_ccw.dae"/>
         </geometry>
         <material name="Blue"/>
@@ -72,13 +72,13 @@
       </inertial>
     </link>
-    <joint name="rotor_0_joint" type="revolute">
+    <joint name="${namespace}/rotor_0_joint" type="revolute">
       <origin xyz="0.13 -0.22 0.023" rpy="0 0 0"/>
-      <parent link="base_link"/>
-      <child link="rotor_0"/>
+      <parent link="${namespace}/base_link"/>
+      <child link="${namespace}/rotor_0"/>
       <axis xyz="0 0 1"/>
       <limit lower="-1e+16" upper="+1e+16" effort="0" velocity="0"/>
     </joint>
     <!-- Gazebo-Specific Properties - Using <gazebo reference="..."> -->
-    <gazebo reference="rotor_0">
+    <gazebo reference="${namespace}/rotor_0">
       <pose>0.13 -0.22 0.023 0 0 0</pose>
       <inertial>
@@ -115,5 +115,5 @@
           <mesh>
             <scale>1 1 1</scale>
-            <uri>$(find ifo_description)/meshes/iris_prop_ccw.dae</uri>
+            <uri>$(find uvify_description)/meshes/iris_prop_ccw.dae</uri>
           </mesh>
         </geometry>
@@ -128,14 +128,14 @@
       <velocity_decay/>
     </gazebo>
-    <gazebo reference="rotor_0_joint">  <!--  Use <gazebo reference="joint_name"> -->
+    <gazebo reference="${namespace}/rotor_0_joint">  <!--  Use <gazebo reference="joint_name"> -->
     </gazebo> <!-- Add Gazebo-specific joint properties here if needed (often not needed for revolute joints) -->
     <!-- ===================================================================== -->
     <!--                               ROTOR 1                                 -->
     <!-- ===================================================================== -->
-    <link name='rotor_1'>
+    <link name='${namespace}/rotor_1'>
       <visual>
         <geometry>
           <!-- <cylinder length="0.01" radius="0.1"/> -->
-          <mesh filename="package://ifo_description/meshes/iris_prop_ccw.dae"/>
+          <mesh filename="package://uvify_description/meshes/iris_prop_ccw.dae"/>
         </geometry>
         <material name="DarkGrey"/>
@@ -146,13 +146,13 @@
       </inertial>
     </link>
-    <joint name="rotor_1_joint" type="revolute">
+    <joint name="${namespace}/rotor_1_joint" type="revolute">
       <origin xyz="-0.13 0.2 0.023" rpy="0 0 0"/>
-      <parent link="base_link"/>
-      <child link="rotor_1"/>
+      <parent link="${namespace}/base_link"/>
+      <child link="${namespace}/rotor_1"/>
       <axis xyz="0 0 1"/>
       <limit lower="-1e+16" upper="+1e+16" effort="0" velocity="0"/>
     </joint>
     <!-- Gazebo-Specific Properties - Using <gazebo reference="..."> -->
-    <gazebo reference="rotor_1">  <!-- Use <gazebo reference="link_name"> -->
+    <gazebo reference="${namespace}/rotor_1">  <!-- Use <gazebo reference="link_name"> -->
       <pose>-0.13 0.2 0.023 0 0 0</pose> <!-- Gazebo-specific pose (if needed) -->
       <inertial>
@@ -189,5 +189,5 @@
           <mesh>
             <scale>1 1 1</scale>
-            <uri>$(find ifo_description)/meshes/iris_prop_ccw.dae</uri>
+            <uri>$(find uvify_description)/meshes/iris_prop_ccw.dae</uri>
           </mesh>
         </geometry>
@@ -202,14 +202,14 @@
       <velocity_decay/>
     </gazebo>
-    <gazebo reference="rotor_1_joint">  <!-- Use <gazebo reference="joint_name"> -->
+    <gazebo reference="${namespace}/rotor_1_joint">  <!-- Use <gazebo reference="joint_name"> -->
     </gazebo> <!-- Add Gazebo-specific joint properties here if needed -->
     <!-- ===================================================================== -->
     <!--                               ROTOR 2                                 -->
     <!-- ===================================================================== -->
-    <link name='rotor_2'>
+    <link name='${namespace}/rotor_2'>
       <visual>
         <geometry>
           <!-- <cylinder length="0.01" radius="0.1"/> -->
-          <mesh filename="package://ifo_description/meshes/iris_prop_cw.dae"/>
+          <mesh filename="package://uvify_description/meshes/iris_prop_cw.dae"/>
         </geometry>
         <material name="Blue"/>
@@ -220,13 +220,13 @@
       </inertial>
     </link>
-    <joint name="rotor_2_joint" type="revolute">
+    <joint name="${namespace}/rotor_2_joint" type="revolute">
       <origin xyz="0.13 0.22 0.023" rpy="0 0 0"/>
-      <parent link="base_link"/>
-      <child link="rotor_2"/>
+      <parent link="${namespace}/base_link"/>
+      <child link="${namespace}/rotor_2"/>
       <axis xyz="0 0 1"/>
       <limit lower="-1e+16" upper="+1e+16" effort="0" velocity="0"/>
     </joint>
     <!-- Gazebo-Specific Properties - Using <gazebo reference="..."> -->
-    <gazebo reference="rotor_2">
+    <gazebo reference="${namespace}/rotor_2">
       <pose>0.13 0.22 0.023 0 0 0</pose>
       <inertial>
@@ -263,5 +263,5 @@
           <mesh>
             <scale>1 1 1</scale>
-            <uri>$(find ifo_description)/meshes/iris_prop_cw.dae</uri>
+            <uri>$(find uvify_description)/meshes/iris_prop_cw.dae</uri>
           </mesh>
         </geometry>
@@ -276,14 +276,14 @@
       <velocity_decay/>
     </gazebo>
-    <gazebo reference="rotor_2_joint">
+    <gazebo reference="${namespace}/rotor_2_joint">
     </gazebo>
     <!-- ===================================================================== -->
     <!--                               ROTOR 3                                 -->
     <!-- ===================================================================== -->
-    <link name='rotor_3'>
+    <link name='${namespace}/rotor_3'>
       <visual>
         <geometry>
           <!-- <cylinder length="0.01" radius="0.1"/> -->
-          <mesh filename="package://ifo_description/meshes/iris_prop_cw.dae"/>
+          <mesh filename="package://uvify_description/meshes/iris_prop_cw.dae"/>
         </geometry>
         <material name="DarkGrey"/>
@@ -294,13 +294,13 @@
       </inertial>
     </link>
-    <joint name="rotor_3_joint" type="revolute">
+    <joint name="${namespace}/rotor_3_joint" type="revolute">
       <origin xyz="-0.13 -0.2 0.023" rpy="0 0 0"/>
-      <parent link="base_link"/>
-      <child link="rotor_3"/>
+      <parent link="${namespace}/base_link"/>
+      <child link="${namespace}/rotor_3"/>
       <axis xyz="0 0 1"/>
       <limit lower="-1e+16" upper="+1e+16" effort="0" velocity="0"/>
     </joint>
     <!-- Gazebo-Specific Properties - Using <gazebo reference="..."> -->
-    <gazebo reference="rotor_3">
+    <gazebo reference="${namespace}/rotor_3">
       <pose>-0.13 -0.2 0.023 0 0 0</pose>
       <inertial>
@@ -337,5 +337,5 @@
           <mesh>
             <scale>1 1 1</scale>
-            <uri>$(find ifo_description)/meshes/iris_prop_cw.dae</uri>
+            <uri>$(find uvify_description)/meshes/iris_prop_cw.dae</uri>
           </mesh>
         </geometry>
@@ -350,5 +350,5 @@
       <velocity_decay/>
     </gazebo>
-    <gazebo reference="rotor_3_joint">
+    <gazebo reference="${namespace}/rotor_3_joint">
     </gazebo>
     <!-- ===================================================================== -->
@@ -356,5 +356,5 @@
     <!-- ===================================================================== -->
     <gazebo>
-      <link name='imu_link'>
+      <link name='${namespace}/imu_link'>
           <pose>0 0 0 0 0 0</pose>
           <inertial>
@@ -371,7 +371,7 @@
           </inertial>
       </link>
-      <joint name='imu_joint' type='revolute'>
-          <child>imu_link</child>
-          <parent>base_link</parent>
+      <joint name='${namespace}/imu_joint' type='revolute'>
+          <child>${namespace}/imu_link</child>
+          <parent>${namespace}/base_link</parent>
           <axis>
           <xyz>1 0 0</xyz>
@@ -396,5 +396,5 @@
       <joint name='gps0_joint' type='fixed'>
         <child>gps0::link</child>
-        <parent>base_link</parent>
+        <parent>${namespace}/base_link</parent>
       </joint>
     </gazebo>
@@ -407,11 +407,11 @@
       <plugin name='rosbag' filename='libgazebo_multirotor_base_plugin.so'>
         <robotNamespace/>
-        <linkName>base_link</linkName>
+        <linkName>${namespace}/base_link</linkName>
         <rotorVelocitySlowdownSim>10</rotorVelocitySlowdownSim>
       </plugin>
       <plugin name='front_right_motor_model' filename='libgazebo_motor_model.so'>
         <robotNamespace/>
-        <jointName>rotor_0_joint</jointName>
-        <linkName>rotor_0</linkName>
+        <jointName>${namespace}/rotor_0_joint</jointName>
+        <linkName>${namespace}/rotor_0</linkName>
         <turningDirection>ccw</turningDirection>
         <timeConstantUp>0.0125</timeConstantUp>
@@ -429,6 +429,6 @@
       <plugin name='back_left_motor_model' filename='libgazebo_motor_model.so'>
         <robotNamespace/>
-        <jointName>rotor_1_joint</jointName>
-        <linkName>rotor_1</linkName>
+        <jointName>${namespace}/rotor_1_joint</jointName>
+        <linkName>${namespace}/rotor_1</linkName>
         <turningDirection>ccw</turningDirection>
         <timeConstantUp>0.0125</timeConstantUp>
@@ -446,6 +446,6 @@
       <plugin name='front_left_motor_model' filename='libgazebo_motor_model.so'>
         <robotNamespace/>
-        <jointName>rotor_2_joint</jointName>
-        <linkName>rotor_2</linkName>
+        <jointName>${namespace}/rotor_2_joint</jointName>
+        <linkName>${namespace}/rotor_2</linkName>
         <turningDirection>cw</turningDirection>
         <timeConstantUp>0.0125</timeConstantUp>
@@ -463,6 +463,6 @@
       <plugin name='back_right_motor_model' filename='libgazebo_motor_model.so'>
         <robotNamespace/>
-        <jointName>rotor_3_joint</jointName>
-        <linkName>rotor_3</linkName>
+        <jointName>${namespace}/rotor_3_joint</jointName>
+        <linkName>${namespace}/rotor_3</linkName>
         <turningDirection>cw</turningDirection>
         <timeConstantUp>0.0125</timeConstantUp>
@@ -619,5 +619,5 @@
       <plugin name='rotors_gazebo_imu_plugin' filename='libgazebo_imu_plugin.so'>
           <robotNamespace/>
-          <linkName>imu_link</linkName>
+          <linkName>${namespace}/imu_link</linkName>
           <imuTopic>/imu</imuTopic>
           <gyroscopeNoiseDensity>0.00018665</gyroscopeNoiseDensity>

File: uvify_description/xacro/iris_depth_camera.xacro (robot description, xacro)
@@ -4,5 +4,5 @@
     <xacro:arg name="mavlink_tcp_port" default="4560" />
     <xacro:arg name="mavlink_udp_port" default="14560" />
-    <xacro:arg name="namespace" default=""/>
+    <xacro:arg name="namespace" default="uvify0"/>
     <xacro:arg name="camera" default="true"/>
     <!-- The following plugin is used to publish the ground truth odometry of the robot
@@ -18,9 +18,9 @@
     </plugin> -->
     <!-- Include base -->
-    <xacro:include filename="$(find ifo_description)/xacro/iris.xacro" />
+    <xacro:include filename="$(find uvify_description)/xacro/iris.xacro" />
     <xacro:iris_base_macro mavlink_tcp_port="$(arg mavlink_tcp_port)" mavlink_udp_port="$(arg mavlink_udp_port)" namespace="$(arg namespace)"/>
     <xacro:if value="$(arg camera)">
-        <xacro:include filename="$(find ifo_description)/xacro/d435.xacro"/>
-        <xacro:sensor_d435 parent="base_link" name="$(arg namespace)/camera" topics_ns="$(arg namespace)" publish_pointcloud="true">
+        <xacro:include filename="$(find uvify_description)/xacro/d435.xacro"/>
+        <xacro:sensor_d435 parent="$(arg namespace)/base_link" name="$(arg namespace)/camera" topics_ns="$(arg namespace)" publish_pointcloud="true">
             <origin xyz="0.12 0 0" rpy="0 0 0" />
         </xacro:sensor_d435>

File: uvify_description/xacro/realsense_d435i.xacro (robot description, xacro)
@@ -27,5 +27,5 @@
       <origin xyz="0 0 0" rpy="1.5707 0 1.5707" />
       <geometry>
-        <mesh filename="package://ifo_description/meshes/d435.dae" />
+        <mesh filename="package://uvify_description/meshes/d435.dae" />
       </geometry>
     </visual>
