Commit message: Added IMU and fixed TF tree

File: uvify_description/xacro/d435.gazebo.xacro (robot description, xacro)
@@ -109,4 +109,85 @@
         <update_rate>90</update_rate>
         <visualize>0</visualize>
+      </sensor>
+    </gazebo>
+    <!-- =================================================================== -->
+    <!--                                 IMU                                 -->
+    <!-- =================================================================== -->
+    <link name="${name}_imu_link"/>
+    <joint name="${name}_imu_joint" type="fixed">
+        <!-- Rotate and translate IMU to be same as real realsense-->
+        <!-- Frame is y DOWN, z forward-->
+      <origin xyz="-0.0051 0.01195 -0.01174" rpy="-1.5707 0 -1.5707" />
+      <parent link="${name}_link"/>
+      <child link="${name}_imu_link"/>
+    </joint>
+    <gazebo reference="${name}_imu_link">
+      <sensor name="imu_sensor" type="imu">
+        <always_on>1</always_on>
+        <update_rate>100.0</update_rate>
+        <topic>${name}/imu</topic>
+        <imu>
+          <angular_velocity>
+            <x>
+              <noise type="gaussian">
+                <mean>0.0</mean>
+                <stddev>0.01</stddev>
+                <bias_mean>0.0</bias_mean>
+                <bias_stddev>0.0001</bias_stddev>
+              </noise>
+            </x>
+            <y>
+              <noise type="gaussian">
+                <mean>0.0</mean>
+                <stddev>0.01</stddev>
+                <bias_mean>0.0</bias_mean>
+                <bias_stddev>0.0001</bias_stddev>
+              </noise>
+            </y>
+            <z>
+              <noise type="gaussian">
+                <mean>0.0</mean>
+                <stddev>0.01</stddev>
+                <bias_mean>0.0</bias_mean>
+                <bias_stddev>0.0001</bias_stddev>
+              </noise>
+            </z>
+          </angular_velocity>
+          <linear_acceleration>
+            <x>
+              <noise type="gaussian">
+                <mean>0.0</mean>
+                <stddev>0.01</stddev>
+                <bias_mean>0.0</bias_mean>
+                <bias_stddev>0.0001</bias_stddev>
+              </noise>
+            </x>
+            <y>
+              <noise type="gaussian">
+                <mean>0.0</mean>
+                <stddev>0.01</stddev>
+                <bias_mean>0.0</bias_mean>
+                <bias_stddev>0.0001</bias_stddev>
+              </noise>
+            </y>
+            <z>
+              <noise type="gaussian">
+                <mean>0.0</mean>
+                <stddev>0.01</stddev>
+                <bias_mean>0.0</bias_mean>
+                <bias_stddev>0.0001</bias_stddev>
+              </noise>
+            </z>
+          </linear_acceleration>
+        </imu>
+        <plugin filename="libgazebo_ros_imu_sensor.so" name="imu_plugin">
+          <robotNamespace></robotNamespace>
+          <topicName>${name}/imu</topicName>
+          <bodyName>${name}_link</bodyName>
+          <updateRateHZ>100.0</updateRateHZ>
+          <xyzOffset>0 0 0</xyzOffset>
+          <rpyOffset>0 0 0</rpyOffset>
+          <frameName>${name}_link</frameName>
+        </plugin>
       </sensor>
     </gazebo>

File: uvify_description/xacro/iris_depth_camera.xacro (robot description, xacro)
@@ -9,13 +9,8 @@
     <xacro:include filename="$(find uvify_description)/xacro/iris.xacro" />
     <xacro:iris_base_macro mavlink_tcp_port="$(arg mavlink_tcp_port)" mavlink_udp_port="$(arg mavlink_udp_port)" namespace="$(arg namespace)"/>
-    <!-- <xacro:if value="$(arg camera)">
+    <xacro:if value="$(arg camera)">
         <xacro:include filename="$(find uvify_description)/xacro/d435.xacro"/>
         <xacro:sensor_d435 parent="$(arg namespace)/base_link" name="$(arg namespace)/camera" topics_ns="$(arg namespace)/camera" publish_pointcloud="true">
             <origin xyz="0.12 0 0" rpy="0 0 0" />
         </xacro:sensor_d435>
-    </xacro:if> -->
-    <xacro:include filename="$(find uvify_description)/xacro/realsense_d435i.xacro"/>
-    <xacro:realsense_d435i parent="$(arg namespace)/base_link" name="$(arg namespace)/camera" topic_ns="$(arg namespace)/camera">
-        <origin xyz="0.12 0 0" rpy="0 0 0" />
-    </xacro:realsense_d435i>
 </robot>
